Commit message: #13 add an extra camera to be able to photograph higher places

File: robutler_description/urdf/robutler.gazebo.xacro (robot description, xacro)
@@ -168,3 +168,37 @@
     </sensor>
   </gazebo>
+<!-- second camera -->
+  <gazebo reference="camera2_rgb_frame">
+    <sensor type="camera" name="Pi Camera">
+      <always_on>true</always_on>
+      <visualize>$(arg camera_visual)</visualize>
+      <camera>
+          <horizontal_fov>1.085595</horizontal_fov>
+          <!-- <horizontal_fov>2.085595</horizontal_fov> -->
+          <image>
+              <width>640</width>
+              <height>480</height>
+              <format>R8G8B8</format>
+          </image>
+          <clip>
+              <near>0.03</near>
+              <far>100</far>
+          </clip>
+      </camera>
+      <plugin name="camera_controller" filename="libgazebo_ros_camera.so">
+        <alwaysOn>true</alwaysOn>
+        <updateRate>30.0</updateRate>
+        <cameraName>camera2</cameraName>
+        <frameName>camera2_rgb_optical_frame</frameName>
+        <imageTopicName>rgb/image_raw</imageTopicName>
+        <cameraInfoTopicName>rgb/camera_info</cameraInfoTopicName>
+        <hackBaseline>0.07</hackBaseline>
+        <distortionK1>0.0</distortionK1>
+        <distortionK2>0.0</distortionK2>
+        <distortionK3>0.0</distortionK3>
+        <distortionT1>0.0</distortionT1>
+        <distortionT2>0.0</distortionT2>
+      </plugin>
+    </sensor>
+  </gazebo>
 </robot>

File: robutler_description/urdf/robutler.urdf.xacro (robot description, xacro)
@@ -185,3 +185,41 @@
   </joint>
   <link name="camera_rgb_optical_frame"/>
+<link name="cylinder_link">
+  <visual>
+    <geometry>
+      <cylinder radius="0.005" length="1"/>
+    </geometry>
+    <origin xyz="0.01 -0.03 0.46" rpy="0 0 0"/>
+  </visual>
+</link>
+<joint name="cylinder_joint" type="fixed">
+  <parent link="base_link"/>
+  <child link="cylinder_link"/>
+  <origin xyz="0.01 -0.03 0.122" rpy="0 0 0"/>
+</joint>
+<joint name="camera2_joint" type="fixed">
+    <origin xyz="0.01 -0.03 1.075" rpy="0 0 0"/>
+    <parent link="base_link"/>
+    <child link="camera2_link"/>
+</joint>
+<link name="camera2_link">
+    <collision>
+      <origin xyz="0.015 -0.03 0.013" rpy="0 0 0"/>
+      <geometry>
+        <box size="0.015 0.030 0.015"/>
+      </geometry>
+    </collision>
+</link>
+<joint name="camera2_rgb_joint" type="fixed">
+    <origin xyz="0.013 0.03 0.009" rpy="0 0 0"/>
+    <parent link="camera2_link"/>
+    <child link="camera2_rgb_frame"/>
+</joint>
+<link name="camera2_rgb_frame"/>
+<joint name="camera2_rgb_optical_joint" type="fixed">
+    <origin xyz="0 0 0" rpy="-1.57 0 -1.57"/>
+    <parent link="camera2_rgb_frame"/>
+    <child link="camera2_rgb_optical_frame"/>
+</joint>
+<link name="camera2_rgb_optical_frame"/>
 </robot>
